File: kicad/WLED_Controller/WLED_Controller.kicad_sch (KiCad schematic)
At the start: 51 parts, among them J1 USB_C_Receptacle_USB2.0, J3 AudioJack, Q1 BC847, Q2 BC847, SW1 SW_RESET, SW2 SW_BOOT, SW3 SW_Push, SW4 SW_Push, SW5 SW_Push, SW6 SW_Push, SW7 SW_Push, U1 ESP32-WROOM-32, U2 CH340C, U3 NCP1117-3.3, U4 TSSP58P38

Commit message: begin creating schematic
Parts:
- removed C13, C14, C15, C16: 100n, Capacitor_SMD:C_0603_1608Metric_Pad1.08x0.95mm_HandSolder, symbol Device:C
- removed SW4, SW5, SW6, SW7: SW_Push, Button_Switch_THT:SW_PUSH_6mm_H13mm, symbol Switch:SW_Push
- added J2, J5: Conn_01x05, GioN_Custom:TerminalBlock_WAGO_236-405_1x05_P5.00mm_45Degree, symbol Connector_Generic:Conn_01x05
- added J6: Conn_01x02, GioN_Custom:TerminalBlock_WAGO_236-402_1x02_P5.00mm_45Degree, symbol Connector_Generic:Conn_01x02
- added JP1, JP4: SolderJumper_3_Open, Jumper:SolderJumper-3_P1.3mm_Open_RoundedPad1.0x1.5mm_NumberLabels, symbol Jumper:SolderJumper_3_Open
- added JP2, JP3: SolderJumper_2_Open, Jumper:SolderJumper-2_P1.3mm_Open_RoundedPad1.0x1.5mm, symbol Jumper:SolderJumper_2_Open
- added Q10, Q3, Q4, Q5, Q6, Q7, Q8, Q9: IRFL4105PBF, Package_TO_SOT_SMD:SOT-223, symbol Transistor_FET:IRF740
- added R13, R14, R23, R24: 100R, Resistor_SMD:R_0603_1608Metric_Pad0.98x0.95mm_HandSolder, symbol Device:R
- added R16, R18, R20, R22, R25, R26, R27, R28: 10k, Resistor_SMD:R_0603_1608Metric_Pad0.98x0.95mm_HandSolder, symbol Device:R
- R15, R17, R19, R21: value 10k -> 100R
Connections:
- net +3.3V: no longer R15.1, R17.1, R19.1, R21.1
- net GND: now also J6.2 (Pin_2), JP1.1 (A), JP4.1 (A), Q10.3 (S), Q3.3 (S), Q4.3 (S), Q5.3 (S), Q6.3 (S), Q7.3 (S), Q8.3 (S), Q9.3 (S), R16.2, R18.2, R20.2, R22.2, R25.2, R26.2, R27.2, R28.2
- net SENSE0: now also J3.2
- net IO12: now reaches U1.14 (IO12)
- net IO21: now reaches U1.33 (IO21)
- net Button1 renamed Button0
- net Button2: no longer names the net of R15.2
- net Button2: now also Q4.1 (G), R16.1; no longer U1.28 (IO17)
- net Button3: no longer names the net of R17.2
- net Button3: now also Q5.1 (G), R18.1; no longer U1.27 (IO16)
- net Button4: no longer names the net of R19.2
- net Button4: now also Q6.1 (G), R20.1; no longer U1.23 (IO15)
- net Button5: no longer names the net of R21.2
- net Button5: now also Q7.1 (G), R22.1; no longer U1.16 (IO13)
- net CS renamed IO5
- net DTA/CTRL renamed IO25
- net MOSI renamed IO23
- net ON renamed IO22
- net RESET renamed IO4
- net SCLK renamed IO18
- net SENSE1 renamed IO14
- net IO14: no longer J3.2
- net SENSE2 renamed IO26
- new net: Q9.1 (G), R23.2, R27.1
- new net: J2.4 (Pin_4), Q9.2 (D)
- new net: Q8.1 (G), R14.2, R26.1
- new net: Q3.1 (G), R13.2, R25.1
- new net: J5.3 (Pin_3), JP2.2 (B), Q5.2 (D)
- new net: J2.3 (Pin_3), JP3.2 (B), Q8.2 (D)
- new net: J5.4 (Pin_4), Q6.2 (D)
- new net: J5.2 (Pin_2), Q4.2 (D)
- new net: J5.5 (Pin_5), JP1.2 (C)
- new net: J2.2 (Pin_2), Q3.2 (D)
- new net: J2.5 (Pin_5), JP4.2 (C)
- new net: Q10.1 (G), R24.2, R28.1
- new net: JP1.3 (B), Q7.2 (D)
- new net: JP4.3 (B), Q10.2 (D)
- new net +24V: J2.1 (Pin_1), J5.1 (Pin_1), J6.1 (Pin_1)
- new net B1: R19.1
- new net B2: R23.1
- new net G1: JP2.1 (A), R17.1
- new net G2: JP3.1 (A), R14.1
- new net IO13: U1.16 (IO13)
- new net IO15: U1.23 (IO15)
- new net IO16: U1.27 (IO16)
- new net IO17: U1.28 (IO17)
- new net R1: R15.1
- new net R2: R13.1
- new net W1: R21.1
- new net W2: R24.1

Commit message: add Microphone
Parts:
- removed J3: AudioJack, GioN_Custom:PG-203JN, symbol GioN_Custom:AudioJack
- added D5: INMP441, GioN_Custom:INMP441_Module, symbol GioN_Custom:INMP441
- added JP5, JP6: SolderJumper_3_Open, Jumper:SolderJumper-3_P1.3mm_Open_RoundedPad1.0x1.5mm_NumberLabels, symbol Jumper:SolderJumper_3_Open
Connections:
- net +24V: now also JP5.3 (B), JP6.3 (B); no longer J2.1 (Pin_1), J5.1 (Pin_1)
- net +3.3V: now also D5.5 (VCC)
- net +5V: now also JP5.1 (A), JP6.1 (A)
- net GND: now also D5.1 (L/R), D5.6 (GND)
- net SENSE0: now also U4.1 (OUT)
- net IO21 renamed MIC_SCK
- net MIC_SCK: now also D5.3 (SCK)
- net IO26 renamed MIC_SD
- net MIC_SD: now also D5.4 (SD)
- net IO5 renamed MIC_WS
- net MIC_WS: now also D5.2 (WS)
- new net: J5.1 (Pin_1), JP5.2 (C)
- new net: J2.1 (Pin_1), JP6.2 (C)

Commit message: Add V1
Parts:
- removed J2, J5: Conn_01x05, GioN_Custom:TerminalBlock_WAGO_236-405_1x05_P5.00mm_45Degree, symbol Connector_Generic:Conn_01x05
- removed JP1, JP4, JP5, JP6: SolderJumper_3_Open, Jumper:SolderJumper-3_P1.3mm_Open_RoundedPad1.0x1.5mm_NumberLabels, symbol Jumper:SolderJumper_3_Open
- removed JP2, JP3: SolderJumper_2_Open, Jumper:SolderJumper-2_P1.3mm_Open_RoundedPad1.0x1.5mm, symbol Jumper:SolderJumper_2_Open
- removed Q10, Q3, Q4, Q5, Q6, Q7, Q8, Q9: IRFL4105PBF, Package_TO_SOT_SMD:SOT-223, symbol Transistor_FET:IRF740
- removed R13, R14, R15, R17, R19, R21, R23, R24: 100R, Resistor_SMD:R_0603_1608Metric_Pad0.98x0.95mm_HandSolder, symbol Device:R
- removed R16, R18, R20, R22, R25, R26, R27, R28: 10k, Resistor_SMD:R_0603_1608Metric_Pad0.98x0.95mm_HandSolder, symbol Device:R
- added C13: 100n, Capacitor_SMD:C_0603_1608Metric_Pad1.08x0.95mm_HandSolder, symbol Device:C
- added J2, J3, J4: Conn_01x03, GioN_Custom:TerminalBlock_WAGO_236-403_1x03_P5.00mm_45Degree, symbol Connector_Generic:Conn_01x03
- added U5: 74HC14, Package_SO:SOIC-14_3.9x8.7mm_P1.27mm, symbol 74xx:74HC14
Connections:
- net +24V is gone; now on net +5V: J6.1 (Pin_1)
- net +5V: now also C13.1, J2.1 (Pin_1), J3.1 (Pin_1), J4.1 (Pin_1), U5.14 (VCC)
- net GND: now also C13.2, J2.3 (Pin_3), J3.3 (Pin_3), J4.3 (Pin_3), U5.7 (GND)
- net at R3.1: now also J1.B5 (CC2); no longer J1.B8 (SBU2)
- net at R5.1: now also J1.A5 (CC1); no longer J1.A8 (SBU1)
- net IO15 renamed LED0
- net LED0: now also U5.1
- net IO16 renamed LED1
- net LED1: now also U5.5
- net IO17 renamed LED2
- net LED2: now also U5.11
- new net: U5.10, U5.13
- new net: U5.2, U5.3
- new net: J3.2 (Pin_2), U5.4
- new net: J4.2 (Pin_2), U5.12
- new net: U5.6, U5.9
- new net: J2.2 (Pin_2), U5.8
Other:
- moved on the sheet: D5, R3, R5

Commit message: Change to WAGO250
Parts:
- J2, J3, J4: footprint GioN_Custom:TerminalBlock_WAGO_236-403_1x03_P5.00mm_45Degree -> GioN_Custom:WAGO_250-203_1x03_P3.50mm
- J6: footprint GioN_Custom:TerminalBlock_WAGO_236-402_1x02_P5.00mm_45Degree -> GioN_Custom:WAGO_250-202_1x02_P3.50mm
Changed lines of the file:
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@@
       (effects (font (size 1.27 1.27)) (justify left))
     )
-    (property "Footprint" "GioN_Custom:TerminalBlock_WAGO_236-403_1x03_P5.00mm_45Degree" (at 266.7 45.72 0)
+    (property "Footprint" "GioN_Custom:WAGO_250-203_1x03_P3.50mm" (at 266.7 45.72 0)
       (effects (font (size 1.27 1.27)) hide)
     )
@@
       (effects (font (size 1.27 1.27)) (justify left))
     )
-    (property "Footprint" "GioN_Custom:TerminalBlock_WAGO_236-403_1x03_P5.00mm_45Degree" (at 266.7 57.15 0)
+    (property "Footprint" "GioN_Custom:WAGO_250-203_1x03_P3.50mm" (at 266.7 57.15 0)
       (effects (font (size 1.27 1.27)) hide)
     )
@@
       (effects (font (size 1.27 1.27)) (justify left))
     )
-    (property "Footprint" "GioN_Custom:TerminalBlock_WAGO_236-402_1x02_P5.00mm_45Degree" (at 125.73 134.62 0)
+    (property "Footprint" "GioN_Custom:WAGO_250-202_1x02_P3.50mm" (at 125.73 134.62 0)
       (effects (font (size 1.27 1.27)) hide)
     )
@@
       (effects (font (size 1.27 1.27)) (justify left))
     )
-    (property "Footprint" "GioN_Custom:TerminalBlock_WAGO_236-403_1x03_P5.00mm_45Degree" (at 266.7 35.56 0)
-      (effects (font (size 1.27 1.27)) hide)
-    )
+    (property "Footprint" "GioN_Custom:WAGO_250-203_1x03_P3.50mm" (at 266.7 35.56 0)
+      (effects (font (size 1.27 1.27)) hide)
+    )
